File: design_files/AST1032.sch (EAGLE design)
At the start: 11 parts, among them J1 SM05B, J2 OLED

Commit message: updated documentation
Parts:
- R2: value 0.0 -> 1.00K; device tinycircuits:AS-ITM-00076 -> tinycircuits:AS-ITM-00003; PARTNO (none) -> AS-ITM-00003; VALUE (none) -> 1.00K
- renumbered J2 to U1
Other:
- note added: "Variant: Standard - R"
- note added: "Wireling 0.96 OLED"
- note removed: "Bio OLED Display"
- note removed: "Variant: Standard"
